Commit message: #20: Gazebo simulation now working

File: kobuki_description/robots/kobuki_kinect.urdf.xacro (robot description, xacro)
@@ -1,11 +1,11 @@
 <?xml version="1.0"?>
 <!--
-    kobuki with Kinect
-    Modified copy from the turtlebot stack
+    Kobuki with Kinect
 -->
 <robot name="kobuki"
        xmlns:sensor="http://playerstage.sourceforge.net/gazebo/xmlschema/#sensor"
        xmlns:controller="http://playerstage.sourceforge.net/gazebo/xmlschema/#controller"
-       xmlns:interface="http://playerstage.sourceforge.net/gazebo/xmlschema/#interface">
+       xmlns:interface="http://playerstage.sourceforge.net/gazebo/xmlschema/#interface"
+       xmlns:xacro="http://ros.org/wiki/xacro">
 	<!-- Included URDF Files -->
   <include filename="$(find kobuki_description)/urdf/kobuki_body.urdf.xacro" />

File: kobuki_description/urdf/gazebo.urdf.xacro (robot description, xacro)
@@ -1,4 +1,8 @@
 <?xml version="1.0"?>
-<robot xmlns:controller="http://playerstage.sourceforge.net/gazebo/xmlschema/#controller" xmlns:interface="http://playerstage.sourceforge.net/gazebo/xmlschema/#interface" xmlns:sensor="http://playerstage.sourceforge.net/gazebo/xmlschema/#sensor" xmlns:xacro="http://ros.org/wiki/xacro" name="turtlebot_gazebo">
+<robot xmlns:controller="http://playerstage.sourceforge.net/gazebo/xmlschema/#controller"
+       xmlns:interface="http://playerstage.sourceforge.net/gazebo/xmlschema/#interface"
+       xmlns:sensor="http://playerstage.sourceforge.net/gazebo/xmlschema/#sensor"
+       xmlns:xacro="http://ros.org/wiki/xacro"
+       name="turtlebot_gazebo">
 <!-- ASUS Xtion PRO camera for simulation -->
 <!-- gazebo_ros_wge100 plugin is in kt2_gazebo_plugins package -->
@@ -87,10 +91,10 @@
       <updateRate>20</updateRate>
       <controller:gazebo_ros_laser name="gazebo_ros_laser_controller" plugin="libgazebo_ros_laser.so">
-	<gaussianNoise>0.005</gaussianNoise>
-	<alwaysOn>true</alwaysOn>
-	<updateRate>20</updateRate>
-	<topicName>scan</topicName>
-	<frameName>laser</frameName>
-	<interface:laser name="gazebo_ros_laser_iface" />
+      	<gaussianNoise>0.005</gaussianNoise>
+      	<alwaysOn>true</alwaysOn>
+      	<updateRate>20</updateRate>
+      	<topicName>scan</topicName>
+      	<frameName>laser</frameName>
+      	<interface:laser name="gazebo_ros_laser_iface" />
       </controller:gazebo_ros_laser>
     </sensor:ray>

File: kobuki_description/urdf/kobuki_body.urdf.xacro (robot description, xacro)
@@ -53,30 +53,33 @@
         <xacro:insert_block name="material_red"/>
       </visual>
-    </link>
+      <collision>
+        <geometry>
+          <cylinder length="${length}" radius="${radius}"/>
+        </geometry>
+        <origin rpy="0 ${pi/2} 0" xyz="0 0 0"/>
+        <xacro:insert_block name="material_red"/>
+      </collision>
+      <inertial>
+        <mass value="0.01" />
+        <origin xyz="0 0 0" />
+        <inertia ixx="0.001" ixy="0.0" ixz="0.0"
+                 iyy="0.001" iyz="0.0"
+                 izz="0.001" />
+      </inertial>
+    </link>
+    <gazebo reference="${name}_link">
+      <material>Gazebo/Black</material>
+    </gazebo>
   </xacro:macro>
   <xacro:macro name="kobuki_body">
-    <!-- needed for navigation stack -->
     <link name="base_footprint">
 <!--       ML: KDL doesn't like inertia in the root link! -->
-<!--       <visual> -->
-<!--         <origin xyz="0 0 0" rpy="0 0 0" /> -->
-<!--         <geometry> -->
-<!-- 	        <box size="0.001 0.001 0.001" /> -->
-<!-- 	      </geometry> -->
-<!-- 	      <xacro:insert_block name="material_red" /> -->
-<!-- 	    </visual> -->
-<!--       <inertial> -->
-<!--         <mass value="0.0001" /> -->
-<!--         <origin xyz="0 0 0" /> -->
-<!--         <inertia ixx="0.0001" ixy="0.0" ixz="0.0" -->
-<!--                  iyy="0.0001" iyz="0.0"  -->
-<!--                  izz="0.0001" /> -->
-<!--       </inertial> -->
-<!--       <collision> -->
-<!-- 	      <origin xyz="0 0 0.017" rpy="0 0 0" /> -->
-<!--   	      <geometry> -->
-<!-- 	          <box size="0.001 0.001 0.001" /> -->
-<!-- 	        </geometry> -->
-<!-- 	    </collision> -->
+      <inertial>
+        <mass value="0.0001" />
+        <origin xyz="0 0 0" />
+        <inertia ixx="0.0001" ixy="0.0" ixz="0.0"
+                 iyy="0.0001" iyz="0.0"
+                 izz="0.0001" />
+      </inertial>
 	  </link>
 		<joint name="base_joint" type="fixed">
@@ -94,9 +97,30 @@
 <!--   TODO: <mesh filename="package://kobuki_description/meshes/kobuki_body.dae"/> -->
 	    </visual>
+      <collision>
+        <geometry>
+          <cylinder length="0.075" radius="0.175"/>
+        </geometry>
+        <origin rpy="0 0 0" xyz="0 0 0.0125"/>
+        <xacro:insert_block name="material_black" />
+      </collision>
+      <inertial>
+        <mass value="0.0001" />
+        <origin xyz="0 0 0" />
+        <inertia ixx="0.0001" ixy="0.0" ixz="0.0"
+                 iyy="0.0001" iyz="0.0"
+                 izz="0.0001" />
+      </inertial>
 	  </link>
-	  <xacro:wheel name="left_wheel"  length="0.020" radius="0.035" off_x="0.00"  off_y="${0.23/2}"  off_z="0.000"   type="continuous">	</xacro:wheel>
-	  <xacro:wheel name="right_wheel" length="0.020" radius="0.035" off_x="0.00"  off_y="-${0.23/2}" off_z="0.000"   type="continuous">	</xacro:wheel>
-	  <xacro:wheel name="front_wheel" length="0.017" radius="0.0175" off_x="0.12"  off_y="0"          off_z="-0.0175" type="fixed">	    </xacro:wheel>
-	  <xacro:wheel name="rear_wheel"  length="0.017" radius="0.0175" off_x="-0.12" off_y="0"          off_z="-0.0175" type="fixed">      </xacro:wheel>
+    <gazebo reference="base_link">
+      <material>Gazebo/Black</material>
+    </gazebo>
+	  <xacro:wheel name="left_wheel"  length="0.020" radius="0.035" off_x="0.00"   off_y="${0.23/2}"  off_z="0.000"
+                 type="continuous">	</xacro:wheel>
+	  <xacro:wheel name="right_wheel" length="0.020" radius="0.035" off_x="0.00"   off_y="-${0.23/2}" off_z="0.000"
+                 type="continuous">	</xacro:wheel>
+	  <xacro:wheel name="front_wheel" length="0.017" radius="0.0175" off_x="0.12"  off_y="0"          off_z="-0.0175"
+                 type="fixed">      </xacro:wheel>
+	  <xacro:wheel name="rear_wheel"  length="0.017" radius="0.0175" off_x="-0.12" off_y="0"          off_z="-0.0175"
+                 type="fixed">        </xacro:wheel>
     <!-- turtlebot topping -->
     <turtlebot_spacer parent="base_link" number="0" x_loc="-0.00254" y_loc="0.1114679" z_loc="0.062992"/>
@@ -255,4 +279,69 @@
       </collision>
     </link>
+  <joint name="base_wall_sensor_joint" type="fixed">
+    <origin xyz="0.09 -0.120 0.042" rpy="0 0 -1.0" />
+    <parent link="base_link"/>
+    <child link="wall_sensor_link" />
+  </joint>
+  <joint name="base_left_cliff_sensor_joint" type="fixed">
+    <origin xyz="0.07 0.14 0.01" rpy="0 1.57079 0" />
+    <parent link="base_link"/>
+    <child link="left_cliff_sensor_link" />
+  </joint>
+  <joint name="base_right_cliff_sensor_joint" type="fixed">
+    <origin xyz="0.07 -0.14 0.01" rpy="0 1.57079 0" />
+    <parent link="base_link"/>
+    <child link="right_cliff_sensor_link" />
+  </joint>
+  <joint name="base_leftfront_cliff_sensor_joint" type="fixed">
+    <origin xyz="0.15 0.04 0.01" rpy="0 1.57079 0" />
+    <parent link="base_link"/>
+    <child link="leftfront_cliff_sensor_link" />
+  </joint>
+  <joint name="base_rightfront_cliff_sensor_joint" type="fixed">
+    <origin xyz="0.15 -0.04 0.01" rpy="0 1.57079 0" />
+    <parent link="base_link"/>
+    <child link="rightfront_cliff_sensor_link" />
+  </joint>
+  <link name="wall_sensor_link">
+    <inertial>
+      <mass value="0.01" />
+      <origin xyz="0 0 0"/>
+      <inertia ixx="0.001" ixy="0.0" ixz="0.0"
+        iyy="0.001" iyz="0.0" izz="0.001" />
+    </inertial>
+  </link>
+  <link name="left_cliff_sensor_link">
+    <inertial>
+      <mass value="0.01" />
+      <origin xyz="0 0 0"/>
+      <inertia ixx="0.001" ixy="0.0" ixz="0.0"
+        iyy="0.001" iyz="0.0" izz="0.001" />
+    </inertial>
+  </link>
+  <link name="right_cliff_sensor_link">
+    <inertial>
+      <mass value="0.01" />
+      <origin xyz="0 0 0"/>
+      <inertia ixx="0.001" ixy="0.0" ixz="0.0"
+        iyy="0.001" iyz="0.0" izz="0.001" />
+    </inertial>
+  </link>
+  <link name="leftfront_cliff_sensor_link">
+    <inertial>
+      <mass value="0.01" />
+      <origin xyz="0 0 0"/>
+      <inertia ixx="1.0" ixy="0.0" ixz="0.0"
+        iyy="0.01" iyz="0.0" izz="0.01" />
+    </inertial>
+  </link>
+  <link name="rightfront_cliff_sensor_link">
+    <inertial>
+      <mass value="0.01" />
+      <origin xyz="0 0 0"/>
+      <inertia ixx="0.001" ixy="0.0" ixz="0.0"
+        iyy="0.001" iyz="0.0" izz="0.001" />
+    </inertial>
+  </link>
     <!-- Simulation sensors TODO-->
     <turtlebot_sim_imu/>
