Commit message: fixes KDL's inertia complain

File: kobuki_description/urdf/kobuki_body.urdf.xacro (robot description, xacro)
@@ -58,5 +58,5 @@
     <!-- needed for navigation stack -->
     <link name="base_footprint">
-<!--       ML: Do we really need visual, inertial and collision here? check turtlebot -->
+<!--       ML: KDL doesn't like inertia in the root link! -->
 <!--       <visual> -->
 <!--         <origin xyz="0 0 0" rpy="0 0 0" /> -->
@@ -66,17 +66,17 @@
 <!-- 	      <xacro:insert_block name="material_red" /> -->
 <!-- 	    </visual> -->
-      <inertial>
-        <mass value="0.0001" />
-        <origin xyz="0 0 0" />
-        <inertia ixx="0.0001" ixy="0.0" ixz="0.0"
-                 iyy="0.0001" iyz="0.0"
-                 izz="0.0001" />
-      </inertial>
-      <collision>
-	      <origin xyz="0 0 0.017" rpy="0 0 0" />
-  	      <geometry>
-	          <box size="0.001 0.001 0.001" />
-	        </geometry>
-	    </collision>
+<!--       <inertial> -->
+<!--         <mass value="0.0001" /> -->
+<!--         <origin xyz="0 0 0" /> -->
+<!--         <inertia ixx="0.0001" ixy="0.0" ixz="0.0" -->
+<!--                  iyy="0.0001" iyz="0.0"  -->
+<!--                  izz="0.0001" /> -->
+<!--       </inertial> -->
+<!--       <collision> -->
+<!-- 	      <origin xyz="0 0 0.017" rpy="0 0 0" /> -->
+<!--   	      <geometry> -->
+<!-- 	          <box size="0.001 0.001 0.001" /> -->
+<!-- 	        </geometry> -->
+<!-- 	    </collision> -->
 	  </link>
 		<joint name="base_joint" type="fixed">
