Commit message: kobuki_description: major updates, restructuring and cleaning

File: kobuki_description/urdf/kobuki.urdf.xacro (robot description, xacro)
@@ -1,6 +1,8 @@
 <?xml version="1.0" ?>
-<robot name="turtlebot_hardware" xmlns:xacro="http://ros.org/wiki/xacro">
+<robot name="kobuki" xmlns:xacro="http://ros.org/wiki/xacro">
   <include filename="$(find kobuki_description)/urdf/common_properties.urdf.xacro"/>
-  <include filename="$(find kobuki_description)/urdf/gazebo.urdf.xacro"/>
+  <include filename="$(find kobuki_description)/urdf/kobuki_gazebo.urdf.xacro"/>
+  <!-- Xacro properties -->
+  <xacro:property name="M_SCALE" value="0.001"/>
   <!-- Xacro macros -->
   <xacro:macro name="wheel" params="name length radius off_x off_y off_z type">
@@ -34,12 +36,25 @@
       </inertial>
     </link>
-<!--     TODO: Needed? -->
-<!--     <gazebo reference="${name}_link"> -->
-<!--       <material>Gazebo/Black</material> -->
-<!--     </gazebo>    -->
+    <gazebo reference="${name}_link">
+      <material>Gazebo/Black</material>
+    </gazebo>
   </xacro:macro>
   <!-- Kobuki -->
   <xacro:macro name="kobuki">
-    <link name="base_footprint"/>
+    <link name="base_footprint">
+      <visual>
+	      <origin xyz="0 0 0" rpy="0 0 0"/>
+	      <geometry>
+	        <box size="0.001 0.001 0.001"/>
+	      </geometry>
+        <xacro:insert_block name="material_black" />
+	    </visual>
+	    <collision>
+	      <origin xyz="0 0 0.035" rpy="0 0 0"/>
+	      <geometry>
+	       <box size="0.001 0.001 0.001"/>
+	      </geometry>
+	    </collision>
+   </link>
 		<joint name="base_joint" type="fixed">
 			<origin xyz="0 0 0.035" rpy="0 0 0" />
@@ -50,5 +65,5 @@
 	    <visual>
 	      <geometry>
-	        <mesh filename="package://kobuki_description/meshes/test/simple_base_new_2.stl" scale="0.001 0.001 0.001"/>
+	        <mesh filename="package://kobuki_description/meshes/kobuki.stl" scale="${M_SCALE} ${M_SCALE} ${M_SCALE}"/>
 	   	  </geometry>
         <origin xyz="0.0 0 0.025" rpy="${M_PI/2} 0 ${M_PI/2}"/>
@@ -62,10 +77,13 @@
       </collision>
       <inertial>
-        <mass value="0.0001" />
-        <origin xyz="0 0 0" />
+        <mass value="2.4"/> <!-- 2.4/2.6 kg for small/big battery pack -->
+        <origin xyz="0 0 0"/>
         <inertia ixx="0.0001" ixy="0.0" ixz="0.0"
                  iyy="0.0001" iyz="0.0"
                  izz="0.0001" />
       </inertial>
+      <gazebo reference="base_link">
+        <material>Gazebo/Black</material>
+      </gazebo>
 	  </link>
 <!--     TODO: Needed? -->
@@ -98,26 +116,50 @@
       </inertial>
     </link>
-	  <joint name="base_cliff_sensor_left_joint" type="fixed">
+	  <joint name="cliff_sensor_left_joint" type="fixed">
 	    <origin xyz="0.07 0.14 0.01" rpy="0 ${M_PI/2} 0" />
 	    <parent link="base_link"/>
-	    <child link="base_cliff_sensor_left_link" />
+	    <child link="cliff_sensor_left_link" />
 	  </joint>
-	  <link name="base_cliff_sensor_left_link"/>
-	  <joint name="base_cliff_sensor_right_joint" type="fixed">
+	  <link name="cliff_sensor_left_link">
+      <inertial>
+        <mass value="0.0001" />
+        <origin xyz="0 0 0" />
+        <inertia ixx="0.0001" ixy="0.0" ixz="0.0"
+                 iyy="0.0001" iyz="0.0"
+                 izz="0.0001" />
+      </inertial>
+    </link>
+	  <joint name="cliff_sensor_right_joint" type="fixed">
 	    <origin xyz="0.07 -0.14 0.01" rpy="0 ${M_PI/2} 0" />
 	    <parent link="base_link"/>
-	    <child link="base_cliff_sensor_right_link" />
+	    <child link="cliff_sensor_right_link" />
 	  </joint>
-    <link name="base_cliff_sensor_right_link"/>
-    <joint name="base_cliff_sensor_front_joint" type="fixed">
+    <link name="cliff_sensor_right_link">
+      <inertial>
+        <mass value="0.0001" />
+        <origin xyz="0 0 0" />
+        <inertia ixx="0.0001" ixy="0.0" ixz="0.0"
+                 iyy="0.0001" iyz="0.0"
+                 izz="0.0001" />
+      </inertial>
+    </link>
+    <joint name="cliff_sensor_front_joint" type="fixed">
       <origin xyz="0.07 -0.14 0.01" rpy="0 ${M_PI/2} 0" />
       <parent link="base_link"/>
-      <child link="base_cliff_sensor_front_link" />
+      <child link="cliff_sensor_front_link" />
     </joint>
-    <link name="base_cliff_sensor_front_link"/>
-    <!-- Simulation sensors TODO-->
-    <turtlebot_sim_kobuki/>
+    <link name="cliff_sensor_front_link">
+      <inertial>
+        <mass value="0.0001" />
+        <origin xyz="0 0 0" />
+        <inertia ixx="0.0001" ixy="0.0" ixz="0.0"
+                 iyy="0.0001" iyz="0.0"
+                 izz="0.0001" />
+      </inertial>
+    </link>
+    <!--  Gazebo additions -->
+    <kobuki_sim/>
+    <kobuki_cliff_sensors/>
     <turtlebot_sim_imu/>
-<!--     <turtlebot_sim_cliff_sensor/> -->
   </xacro:macro>
 </robot>

File: kobuki_description/urdf/turtlebot2_stack.urdf.xacro (robot description, xacro)
@@ -1,3 +1,6 @@
 <?xml version="1.0"?>
+<!--
+  Turtlebot 2 stack (plates + poles)
+ -->
 <robot name="turtlebot2_stack" xmlns:xacro="http://ros.org/wiki/xacro">
   <include filename="$(find kobuki_description)/urdf/common_properties.urdf.xacro"/>
@@ -15,5 +18,5 @@
         <origin xyz="0 0 0" rpy="${M_PI/2} 0 ${M_PI/2}"/>
         <geometry>
-          <mesh filename="package://kobuki_description/meshes/high_res_stl/poll_1st.stl" scale="${M_SCALE} ${M_SCALE} ${M_SCALE}"/>
+          <mesh filename="package://kobuki_description/meshes/turtlebot2_stack/high_res/poll_1st.stl" scale="${M_SCALE} ${M_SCALE} ${M_SCALE}"/>
         </geometry>
         <xacro:insert_block name="material_light_grey"/>
@@ -44,5 +47,5 @@
         <origin xyz="0 0 0" rpy="${-M_PI/2} 0 0"/>
         <geometry>
-          <mesh filename="package://kobuki_description/meshes/high_res_stl/poll_2nd.stl" scale="${M_SCALE} ${M_SCALE} ${M_SCALE}"/>
+          <mesh filename="package://kobuki_description/meshes/turtlebot2_stack/high_res/poll_2nd.stl" scale="${M_SCALE} ${M_SCALE} ${M_SCALE}"/>
         </geometry>
         <xacro:insert_block name="material_light_grey"/>
@@ -53,5 +56,4 @@
           <cylinder length="0.0608" radius=".006"/>
         </geometry>
-        <xacro:insert_block name="material_light_grey"/>
       </collision>
       <inertial>
@@ -74,5 +76,5 @@
         <origin xyz=" 0 0 0" rpy="${M_PI/2} 0 ${M_PI/2}"/>
         <geometry>
-          <mesh filename="package://kobuki_description/meshes/high_res_stl/poll_3rd.stl" scale="${M_SCALE} ${M_SCALE} ${M_SCALE}"/>
+          <mesh filename="package://kobuki_description/meshes/turtlebot2_stack/high_res/poll_3rd.stl" scale="${M_SCALE} ${M_SCALE} ${M_SCALE}"/>
         </geometry>
         <xacro:insert_block name="material_light_grey"/>
@@ -83,5 +85,4 @@
           <cylinder length="0.2032" radius=".006"/>
         </geometry>
-        <xacro:insert_block name="material_light_grey"/>
       </collision>
       <inertial>
@@ -111,5 +112,5 @@
         <origin xyz=" 0 0 0 " rpy="0 0 0"/>
         <geometry>
-          <mesh filename="package://kobuki_description/meshes/high_res_stl/poll_kinect.stl" scale="${M_SCALE} ${M_SCALE} ${M_SCALE}"/>
+          <mesh filename="package://kobuki_description/meshes/turtlebot2_stack/high_res/poll_kinect.stl" scale="${M_SCALE} ${M_SCALE} ${M_SCALE}"/>
         </geometry>
         <xacro:insert_block name="material_light_grey"/>
@@ -120,5 +121,4 @@
           <cylinder length="0.008585" radius="0.001111"/>
         </geometry>
-        <xacro:insert_block name="material_light_grey" />
       </collision>
     </link>
@@ -133,7 +133,7 @@
     <stack_bottom_pole parent="${parent}" number="5" x_loc="-0.055" y_loc="-0.120" z_loc="0.0534"/>
 		<joint name="plate_bottom_joint" type="fixed">
-		  <origin xyz="0.0 0.0  0.1026" rpy="0 0 0" />
+		  <origin xyz="0.0 0.0  0.1026" rpy="0 0 0"/>
 		  <parent link="${parent}"/>
-		  <child link="plate_bottom_link" />
+		  <child link="plate_bottom_link"/>
 		</joint>
 		<link name="plate_bottom_link">
@@ -141,7 +141,7 @@
 		    <origin xyz="0 0 0" rpy="${M_PI/2} 0 ${M_PI/2}"/>
 		    <geometry>
-		      <mesh filename="package://kobuki_description/meshes/high_res_stl/stack_1st.stl" scale="${M_SCALE} ${M_SCALE} ${M_SCALE}"/>
-		    </geometry>
-        <xacro:insert_block name="material_light_grey" />
+		      <mesh filename="package://kobuki_description/meshes/turtlebot2_stack/high_res/stack_1st.stl" scale="${M_SCALE} ${M_SCALE} ${M_SCALE}"/>
+		    </geometry>
+        <xacro:insert_block name="material_light_grey"/>
 		  </visual>
 		  <collision>
@@ -150,5 +150,5 @@
 		      <box size="0.26727 0.345 0.006"/>
 		    </geometry>
-        <xacro:insert_block name="material_light_grey" />
+        <xacro:insert_block name="material_light_grey"/>
 		  </collision>
       <inertial>
@@ -173,7 +173,7 @@
 		    <origin xyz="0 0 0" rpy="${M_PI/2} 0 ${M_PI/2}"/>
 		    <geometry>
-		      <mesh filename="package://kobuki_description/meshes/high_res_stl/stack_2nd.stl" scale="${M_SCALE} ${M_SCALE} ${M_SCALE}"/>
-		    </geometry>
-        <xacro:insert_block name="material_grey" />
+		      <mesh filename="package://kobuki_description/meshes/turtlebot2_stack/high_res/stack_2nd.stl" scale="${M_SCALE} ${M_SCALE} ${M_SCALE}"/>
+		    </geometry>
+        <xacro:insert_block name="material_light_grey"/>
 		  </visual>
 		  <collision>
@@ -182,5 +182,4 @@
 		      <box size="0.31454 0.345 0.006"/>
 		    </geometry>
-        <xacro:insert_block name="material_grey" />
 		  </collision>
       <inertial>
@@ -205,7 +204,7 @@
         <origin xyz="0 0 0" rpy="${M_PI/2} 0 ${M_PI/2}"/>
 		    <geometry>
-		      <mesh filename="package://kobuki_description/meshes/high_res_stl/stack_3rd.stl" scale="${M_SCALE} ${M_SCALE} ${M_SCALE}"/>
-		    </geometry>
-        <xacro:insert_block name="material_grey" />
+		      <mesh filename="package://kobuki_description/meshes/turtlebot2_stack/high_res/stack_3rd.stl" scale="${M_SCALE} ${M_SCALE} ${M_SCALE}"/>
+		    </geometry>
+        <xacro:insert_block name="material_light_grey"/>
 		  </visual>
 		  <collision>
@@ -214,5 +213,4 @@
 		      <box size="0.233502 0.314845 0.006401"/>
 		    </geometry>
-        <xacro:insert_block name="material_grey" />
 		  </collision>
       <inertial>

Commit message: match the create convention for base link at the bottom of the base.

File: kobuki_description/urdf/kobuki.urdf.xacro (robot description, xacro)
@@ -58,5 +58,5 @@
    </link>
 		<joint name="base_joint" type="fixed">
-			<origin xyz="0 0 0.035" rpy="0 0 0" />
+			<origin xyz="0 0 0.017" rpy="0 0 0" />
 			<parent link="base_footprint"/>
 			<child link="base_link" />
@@ -67,5 +67,5 @@
 	        <mesh filename="package://kobuki_description/meshes/kobuki.stl" scale="${M_SCALE} ${M_SCALE} ${M_SCALE}"/>
 	   	  </geometry>
-        <origin xyz="0.0 0 0.025" rpy="${M_PI/2} 0 ${M_PI/2}"/>
+        <origin xyz="0.0 0 0.043" rpy="${M_PI/2} 0 ${M_PI/2}"/>
         <xacro:insert_block name="material_black" />
 	    </visual>
@@ -91,11 +91,11 @@
 <!--       <material>Gazebo/Black</material> -->
 <!--     </gazebo>         -->
-	  <xacro:wheel name="wheel_left"  length="0.0206" radius="0.0350" off_x="0.00"   off_y="${0.23/2}"  off_z="0.000"
+	  <xacro:wheel name="wheel_left"  length="0.0206" radius="0.0350" off_x="0.00"   off_y="${0.23/2}"  off_z="0.018"
                  type="continuous">	</xacro:wheel>
-	  <xacro:wheel name="wheel_right" length="0.0206" radius="0.0350" off_x="0.00"   off_y="-${0.23/2}" off_z="0.000"
+	  <xacro:wheel name="wheel_right" length="0.0206" radius="0.0350" off_x="0.00"   off_y="-${0.23/2}" off_z="0.018"
                  type="continuous">	</xacro:wheel>
-	  <xacro:wheel name="caster_front" length="0.0176" radius="0.0170" off_x="0.115"  off_y="0"          off_z="-0.0180"
+	  <xacro:wheel name="caster_front" length="0.0176" radius="0.0170" off_x="0.115"  off_y="0"          off_z="-0.0000"
                  type="fixed">      </xacro:wheel>
-	  <xacro:wheel name="caster_back"  length="0.0176" radius="0.0170" off_x="-0.135" off_y="0"          off_z="-0.0160"
+	  <xacro:wheel name="caster_back"  length="0.0176" radius="0.0170" off_x="-0.135" off_y="0"          off_z="0.0020"
                  type="fixed">      </xacro:wheel>
     <!-- Kobuki's sensors -->
@@ -103,5 +103,5 @@
     <joint name="gyro_joint" type="fixed">
       <axis xyz="0 1 0"/>
-      <origin xyz="0 0 0.04" rpy="0 0 0"/>
+      <origin xyz="0 0 0.058" rpy="0 0 0"/>
       <parent link="base_link"/>
       <child link="gyro_link"/>
@@ -117,5 +117,5 @@
     </link>
 	  <joint name="cliff_sensor_left_joint" type="fixed">
-	    <origin xyz="0.07 0.14 0.01" rpy="0 ${M_PI/2} 0" />
+	    <origin xyz="0.07 0.14 0.028" rpy="0 ${M_PI/2} 0" />
 	    <parent link="base_link"/>
 	    <child link="cliff_sensor_left_link" />
@@ -131,5 +131,5 @@
     </link>
 	  <joint name="cliff_sensor_right_joint" type="fixed">
-	    <origin xyz="0.07 -0.14 0.01" rpy="0 ${M_PI/2} 0" />
+	    <origin xyz="0.07 -0.14 0.028" rpy="0 ${M_PI/2} 0" />
 	    <parent link="base_link"/>
 	    <child link="cliff_sensor_right_link" />
@@ -145,5 +145,5 @@
     </link>
     <joint name="cliff_sensor_front_joint" type="fixed">
-      <origin xyz="0.07 -0.14 0.01" rpy="0 ${M_PI/2} 0" />
+      <origin xyz="0.07 -0.14 0.028" rpy="0 ${M_PI/2} 0" />
       <parent link="base_link"/>
       <child link="cliff_sensor_front_link" />

Commit message: updates some poses for the use of the new collada meshes (plus some cleaning)

File: kobuki_description/urdf/kobuki.urdf.xacro (robot description, xacro)
@@ -5,74 +5,45 @@
   <!-- Xacro properties -->
   <xacro:property name="M_SCALE" value="0.001"/>
-  <!-- Xacro macros -->
-  <xacro:macro name="wheel" params="name length radius off_x off_y off_z type">
-    <joint name="${name}_joint" type="${type}">
-      <parent link="base_link"/>
-      <child link="${name}_link"/>
-      <origin rpy="${-M_PI/2} 0 0" xyz="${off_x} ${off_y} ${off_z}"/>
-      <axis xyz="0 0 1"/>
-    </joint>
-    <link name="${name}_link">
-      <visual>
-        <geometry>
-          <cylinder length="${length}" radius="${radius}"/>
-        </geometry>
-        <origin rpy="0 0 0" xyz="0 0 0"/>
-        <xacro:insert_block name="material_dark_grey"/>
-      </visual>
-      <collision>
-        <geometry>
-          <cylinder length="${length}" radius="${radius}"/>
-        </geometry>
-        <origin rpy="0 0 0" xyz="0 0 0"/>
-        <xacro:insert_block name="material_dark_grey"/>
-      </collision>
-      <inertial>
-        <mass value="0.01" />
-        <origin xyz="0 0 0" />
-        <inertia ixx="0.001" ixy="0.0" ixz="0.0"
-                 iyy="0.001" iyz="0.0"
-                 izz="0.001" />
-      </inertial>
-    </link>
-    <gazebo reference="${name}_link">
-      <material>Gazebo/Black</material>
-    </gazebo>
-  </xacro:macro>
   <!-- Kobuki -->
   <xacro:macro name="kobuki">
     <link name="base_footprint">
       <visual>
-	      <origin xyz="0 0 0" rpy="0 0 0"/>
-	      <geometry>
-	        <box size="0.001 0.001 0.001"/>
-	      </geometry>
+        <origin xyz="0 0 0" rpy="0 0 0"/>
+        <geometry>
+          <box size="0.001 0.001 0.001"/>
+        </geometry>
         <xacro:insert_block name="material_black" />
-	    </visual>
-	    <collision>
-	      <origin xyz="0 0 0.035" rpy="0 0 0"/>
-	      <geometry>
-	       <box size="0.001 0.001 0.001"/>
-	      </geometry>
-	    </collision>
-   </link>
-		<joint name="base_joint" type="fixed">
-			<origin xyz="0 0 0.017" rpy="0 0 0" />
-			<parent link="base_footprint"/>
-			<child link="base_link" />
-		</joint>
-	  <link name="base_link">
-	    <visual>
-	      <geometry>
-	        <mesh filename="package://kobuki_description/meshes/kobuki.stl" scale="${M_SCALE} ${M_SCALE} ${M_SCALE}"/>
-	   	  </geometry>
-        <origin xyz="0.0 0 0.043" rpy="${M_PI/2} 0 ${M_PI/2}"/>
-        <xacro:insert_block name="material_black" />
-	    </visual>
+      </visual>
+      <collision>
+        <origin xyz="0 0 0.035" rpy="0 0 0"/>
+        <geometry>
+         <box size="0.001 0.001 0.001"/>
+        </geometry>
+      </collision>
+    </link>
+    <joint name="base_bottom_joint" type="fixed">
+      <origin xyz="0 0 0.0102" rpy="0 0 0" />
+      <parent link="base_footprint"/>
+      <child link="base_bottom_link" />
+    </joint>
+    <link name="base_bottom_link"/>
+    <joint name="base_joint" type="fixed">
+      <origin xyz="0 0 0.0352" rpy="0 0 0" />
+      <parent link="base_footprint"/>
+      <child link="base_link" />
+    </joint>
+    <link name="base_link">
+      <visual>
+        <geometry>
+          <mesh filename="package://kobuki_description/meshes/base.dae" scale="${M_SCALE} ${M_SCALE} ${M_SCALE}"/>
+        </geometry>
+        <origin xyz="0.0 0 0.02969" rpy="${M_PI/2} 0 ${M_PI/2}"/>
+        <xacro:insert_block name="material_black"/>
+      </visual>
       <collision>
         <geometry>
           <cylinder length="0.10938" radius="0.175615"/>
         </geometry>
-        <origin xyz="0.0 0.0 0.03469" rpy="0 0 0"/>
+        <origin xyz="0.0 0.0 0.02969" rpy="0 0 0"/>
       </collision>
       <inertial>
@@ -86,17 +57,61 @@
         <material>Gazebo/Black</material>
       </gazebo>
-	  </link>
-<!--     TODO: Needed? -->
-<!--     <gazebo reference="base_link"> -->
-<!--       <material>Gazebo/Black</material> -->
-<!--     </gazebo>         -->
-	  <xacro:wheel name="wheel_left"  length="0.0206" radius="0.0350" off_x="0.00"   off_y="${0.23/2}"  off_z="0.018"
-                 type="continuous">	</xacro:wheel>
-	  <xacro:wheel name="wheel_right" length="0.0206" radius="0.0350" off_x="0.00"   off_y="-${0.23/2}" off_z="0.018"
-                 type="continuous">	</xacro:wheel>
-	  <xacro:wheel name="caster_front" length="0.0176" radius="0.0170" off_x="0.115"  off_y="0"          off_z="-0.0000"
-                 type="fixed">      </xacro:wheel>
-	  <xacro:wheel name="caster_back"  length="0.0176" radius="0.0170" off_x="-0.135" off_y="0"          off_z="0.0020"
-                 type="fixed">      </xacro:wheel>
+    </link>
+    <joint name="wheel_left_joint" type="continuous">
+      <parent link="base_link"/>
+      <child link="wheel_left_link"/>
+      <origin xyz="0.00 ${0.23/2} 0.00" rpy="${-M_PI/2} 0 0"/>
+      <axis xyz="0 0 1"/>
+    </joint>
+    <link name="wheel_left_link">
+      <visual>
+        <geometry>
+          <mesh filename="package://kobuki_description/meshes/wheel.dae" scale="${M_SCALE} ${M_SCALE} ${M_SCALE}"/>
+        </geometry>
+        <origin xyz="0 0 0" rpy="0 ${M_PI/2} 0"/>
+        <xacro:insert_block name="material_black"/>
+      </visual>
+      <collision>
+        <geometry>
+          <cylinder length="0.0206" radius="0.0352"/>
+        </geometry>
+        <origin rpy="0 0 0" xyz="0 0 0"/>
+      </collision>
+      <inertial>
+        <mass value="0.01" />
+        <origin xyz="0 0 0" />
+        <inertia ixx="0.001" ixy="0.0" ixz="0.0"
+                 iyy="0.001" iyz="0.0"
+                 izz="0.001" />
+      </inertial>
+    </link>
+    <joint name="wheel_right_joint" type="continuous">
+      <parent link="base_link"/>
+      <child link="wheel_right_link"/>
+      <origin xyz="0.00 -${0.23/2} 0.00" rpy="${-M_PI/2} 0 0"/>
+      <axis xyz="0 0 1"/>
+    </joint>
+    <link name="wheel_right_link">
+      <visual>
+        <geometry>
+          <mesh filename="package://kobuki_description/meshes/wheel.dae" scale="${M_SCALE} ${M_SCALE} ${M_SCALE}"/>
+        </geometry>
+        <origin xyz="0 0 0" rpy="0 ${M_PI/2} 0"/>
+        <xacro:insert_block name="material_black"/>
+      </visual>
+      <collision>
+        <geometry>
+          <cylinder length="0.0206" radius="0.0350"/>
+        </geometry>
+        <origin rpy="0 0 0" xyz="0 0 0"/>
+      </collision>
+      <inertial>
+        <mass value="0.01" />
+        <origin xyz="0 0 0" />
+        <inertia ixx="0.001" ixy="0.0" ixz="0.0"
+                 iyy="0.001" iyz="0.0"
+                 izz="0.001" />
+      </inertial>
+    </link>
     <!-- Kobuki's sensors -->
     <!-- TODO: Check placement! -->

Commit message: Move back to turtlebot convention, base link at the base of the mould.

File: kobuki_description/urdf/kobuki.urdf.xacro (robot description, xacro)
@@ -22,12 +22,15 @@
       </collision>
     </link>
-    <joint name="base_bottom_joint" type="fixed">
+     <!--
+       Base link is set at the bottom of the base mould.
+       This is done to be compatible with the way base link
+       was configured for turtlebot 1. Refer to
+       https://github.com/turtlebot/turtlebot/issues/40
+       To put the base link at the more oft used wheel
+       axis, set the z-distance from the base_footprint
+       to 0.352.
+      -->
+    <joint name="base_joint" type="fixed">
       <origin xyz="0 0 0.0102" rpy="0 0 0" />
-      <parent link="base_footprint"/>
-      <child link="base_bottom_link" />
-    </joint>
-    <link name="base_bottom_link"/>
-    <joint name="base_joint" type="fixed">
-      <origin xyz="0 0 0.0352" rpy="0 0 0" />
       <parent link="base_footprint"/>
       <child link="base_link" />
@@ -38,5 +41,5 @@
           <mesh filename="package://kobuki_description/meshes/base.dae" scale="${M_SCALE} ${M_SCALE} ${M_SCALE}"/>
         </geometry>
-        <origin xyz="0.0 0 0.02969" rpy="${M_PI/2} 0 ${M_PI/2}"/>
+        <origin xyz="0.0 0 0.05469" rpy="${M_PI/2} 0 ${M_PI/2}"/>
         <xacro:insert_block name="material_black"/>
       </visual>
@@ -45,5 +48,5 @@
           <cylinder length="0.10938" radius="0.175615"/>
         </geometry>
-        <origin xyz="0.0 0.0 0.02969" rpy="0 0 0"/>
+        <origin xyz="0.0 0.0 0.05469" rpy="0 0 0"/>
       </collision>
       <inertial>
@@ -61,5 +64,5 @@
       <parent link="base_link"/>
       <child link="wheel_left_link"/>
-      <origin xyz="0.00 ${0.23/2} 0.00" rpy="${-M_PI/2} 0 0"/>
+      <origin xyz="0.00 ${0.23/2} 0.0250" rpy="${-M_PI/2} 0 0"/>
       <axis xyz="0 0 1"/>
     </joint>
@@ -89,5 +92,5 @@
       <parent link="base_link"/>
       <child link="wheel_right_link"/>
-      <origin xyz="0.00 -${0.23/2} 0.00" rpy="${-M_PI/2} 0 0"/>
+      <origin xyz="0.00 -${0.23/2} 0.0250" rpy="${-M_PI/2} 0 0"/>
       <axis xyz="0 0 1"/>
     </joint>
@@ -160,5 +163,5 @@
     </link>
     <joint name="cliff_sensor_front_joint" type="fixed">
-      <origin xyz="0.07 -0.14 0.028" rpy="0 ${M_PI/2} 0" />
+      <origin xyz="0.18 0.00 0.028" rpy="0 ${M_PI/2} 0" />
       <parent link="base_link"/>
       <child link="cliff_sensor_front_link" />
