Commit message: updated urdf and mesh

File: kobuki_description/urdf/kobuki.urdf.xacro (robot description, xacro)
@@ -13,20 +13,6 @@
   <!-- Kobuki -->
   <xacro:macro name="kobuki">
-    <link name="base_footprint">
-      <visual>
-        <origin xyz="0 0 0" rpy="0 0 0"/>
-        <geometry>
-          <box size="0.001 0.001 0.001"/>
-        </geometry>
-        <xacro:insert_block name="material_black" />
-      </visual>
-      <collision>
-        <origin xyz="0 0 0.035" rpy="0 0 0"/>
-        <geometry>
-         <box size="0.001 0.001 0.001"/>
-        </geometry>
-      </collision>
-    </link>
-     <!--
+    <link name="base_footprint"/>
+    <!--
        Base link is set at the bottom of the base mould.
        This is done to be compatible with the way base link
@@ -45,14 +31,14 @@
       <visual>
         <geometry>
-          <mesh filename="package://kobuki_description/meshes/base.dae" scale="${M_SCALE} ${M_SCALE} ${M_SCALE}"/>
-        </geometry>
-        <origin xyz="0.0 0 0.05469" rpy="${M_PI/2} 0 ${M_PI/2}"/>
-        <xacro:insert_block name="material_black"/>
+          <!-- new mesh -->
+          <mesh filename="package://kobuki_description/meshes/main_body.dae" />
+        </geometry>
+        <origin xyz="0.001 0 0.05199" rpy="0 0 0"/>
       </visual>
       <collision>
         <geometry>
-          <cylinder length="0.10938" radius="0.175615"/>
-        </geometry>
-        <origin xyz="0.0 0.0 0.05469" rpy="0 0 0"/>
+          <cylinder length="0.10938" radius="0.176"/>
+        </geometry>
+        <origin xyz="0.0 0 0.05949" rpy="0 0 0"/>
       </collision>
       <inertial>
@@ -63,7 +49,4 @@
                  izz="0.0001" />
       </inertial>
-      <gazebo reference="base_link">
-        <material>Gazebo/Black</material>
-      </gazebo>
     </link>
     <joint name="wheel_left_joint" type="continuous">
@@ -76,8 +59,7 @@
       <visual>
         <geometry>
-          <mesh filename="package://kobuki_description/meshes/wheel.dae" scale="${M_SCALE} ${M_SCALE} ${M_SCALE}"/>
-        </geometry>
-        <origin xyz="0 0 0" rpy="0 ${M_PI/2} 0"/>
-        <xacro:insert_block name="material_black"/>
+          <mesh filename="package://kobuki_description/meshes/wheel.dae"/>
+        </geometry>
+        <origin xyz="0 0 0" rpy="0 0 0"/>
       </visual>
       <collision>
@@ -104,8 +86,7 @@
       <visual>
         <geometry>
-          <mesh filename="package://kobuki_description/meshes/wheel.dae" scale="${M_SCALE} ${M_SCALE} ${M_SCALE}"/>
-        </geometry>
-        <origin xyz="0 0 0" rpy="0 ${M_PI/2} 0"/>
-        <xacro:insert_block name="material_black"/>
+          <mesh filename="package://kobuki_description/meshes/wheel.dae"/>
+        </geometry>
+        <origin xyz="0 0 0" rpy="0 0 0"/>
       </visual>
       <collision>
@@ -123,9 +104,48 @@
       </inertial>
     </link>
+    <joint name="caster_front_joint" type="fixed">
+      <parent link="base_link"/>
+      <child link="caster_front_link"/>
+      <origin xyz="0.115 0.0 0.007" rpy="${-M_PI/2} 0 0"/>
+    </joint>
+    <link name="caster_front_link">
+      <collision>
+        <geometry>
+          <cylinder length="0.0176" radius="0.017"/>
+        </geometry>
+        <origin rpy="0 0 0" xyz="0 0 0"/>
+      </collision>
+      <inertial>
+        <mass value="0.01" />
+        <origin xyz="0 0 0" />
+        <inertia ixx="0.001" ixy="0.0" ixz="0.0"
+                 iyy="0.001" iyz="0.0"
+                 izz="0.001" />
+      </inertial>
+    </link>
+    <joint name="caster_back_joint" type="fixed">
+      <parent link="base_link"/>
+      <child link="caster_back_link"/>
+      <origin xyz="-0.135 0.0 0.009" rpy="${-M_PI/2} 0 0"/>
+    </joint>
+    <link name="caster_back_link">
+      <collision>
+        <geometry>
+          <cylinder length="0.0176" radius="0.017"/>
+        </geometry>
+        <origin rpy="0 0 0" xyz="0 0 0"/>
+      </collision>
+      <inertial>
+        <mass value="0.01" />
+        <origin xyz="0 0 0" />
+        <inertia ixx="0.001" ixy="0.0" ixz="0.0"
+                 iyy="0.001" iyz="0.0"
+                 izz="0.001" />
+      </inertial>
+    </link>
     <!-- Kobuki's sensors -->
-    <!-- TODO: Check placement! -->
     <joint name="gyro_joint" type="fixed">
       <axis xyz="0 1 0"/>
-      <origin xyz="0 0 0.058" rpy="0 0 0"/>
+      <origin xyz="0.056 0.062 0.0202" rpy="0 0 0"/>
       <parent link="base_link"/>
       <child link="gyro_link"/>
@@ -141,5 +161,5 @@
     </link>
 	  <joint name="cliff_sensor_left_joint" type="fixed">
-	    <origin xyz="0.07 0.14 0.028" rpy="0 ${M_PI/2} 0" />
+	    <origin xyz="0.08734 0.13601 0.0214" rpy="0 ${M_PI/2} 0" />
 	    <parent link="base_link"/>
 	    <child link="cliff_sensor_left_link" />
@@ -155,5 +175,5 @@
     </link>
 	  <joint name="cliff_sensor_right_joint" type="fixed">
-	    <origin xyz="0.07 -0.14 0.028" rpy="0 ${M_PI/2} 0" />
+	    <origin xyz="0.085 -0.13601 0.0214" rpy="0 ${M_PI/2} 0" />
 	    <parent link="base_link"/>
 	    <child link="cliff_sensor_right_link" />
@@ -169,5 +189,5 @@
     </link>
     <joint name="cliff_sensor_front_joint" type="fixed">
-      <origin xyz="0.18 0.00 0.028" rpy="0 ${M_PI/2} 0" />
+      <origin xyz="0.156 0.00 0.0214" rpy="0 ${M_PI/2} 0" />
       <parent link="base_link"/>
       <child link="cliff_sensor_front_link" />
@@ -184,6 +204,7 @@
     <!--  Gazebo additions -->
     <kobuki_sim/>
+    <kobuki_bumpers/>
     <kobuki_cliff_sensors/>
-    <turtlebot_sim_imu/>
+    <kobuki_sim_imu/>
   </xacro:macro>
 </robot>

File: kobuki_description/urdf/kobuki_gazebo.urdf.xacro (robot description, xacro)
@@ -4,17 +4,74 @@
        xmlns:sensor="http://playerstage.sourceforge.net/gazebo/xmlschema/#sensor"
        xmlns:xacro="http://ros.org/wiki/xacro"
-       name="turtlebot_gazebo">
+       name="kobuki_gazebo">
+<xacro:macro name="kobuki_bumpers">
+  <gazebo reference="base_link">
+    <sensor:contact name="bumpers">
+      <geom>base_footprint_geom_base_link</geom>
+      <topic>bumpers</topic>
+      <alwaysOn>true</alwaysOn>
+      <updateRate>50</updateRate>
+    </sensor:contact>
+  </gazebo>
+</xacro:macro>
+<xacro:macro name="kobuki_cliff_sensors">
+  <gazebo reference="cliff_sensor_left_link">
+    <sensor:ray name="cliff_sensor_left">
+      <alwaysOn>true</alwaysOn>
+      <updateRate>50</updateRate>
+      <rayCount>50</rayCount>
+      <rangeCount>1</rangeCount>
+      <resRange>1.0</resRange>
+      <minAngle>-0.04361</minAngle>
+      <maxAngle>0.04361</maxAngle>
+      <minRange>0.01</minRange>
+      <maxRange>0.15</maxRange>
+      <displayRays>true</displayRays>
+    </sensor:ray>
+  </gazebo>
+  <gazebo reference="cliff_sensor_right_link">
+    <sensor:ray name="cliff_sensor_right">
+      <alwaysOn>true</alwaysOn>
+      <updateRate>50</updateRate>
+      <rayCount>50</rayCount>
+      <rangeCount>1</rangeCount>
+      <resRange>1.0</resRange>
+      <minAngle>-2.5</minAngle>
+      <maxAngle>2.5</maxAngle>
+      <minRange>0.01</minRange>
+      <maxRange>0.15</maxRange>
+      <displayRays>true</displayRays>
+    </sensor:ray>
+  </gazebo>
+  <gazebo reference="cliff_sensor_front_link">
+    <sensor:ray name="cliff_sensor_front">
+      <alwaysOn>true</alwaysOn>
+      <updateRate>50</updateRate>
+      <rayCount>50</rayCount>
+      <rangeCount>1</rangeCount>
+      <resRange>1.0</resRange>
+      <minAngle>-2.5</minAngle>
+      <maxAngle>2.5</maxAngle>
+      <minRange>0.01</minRange>
+      <maxRange>0.15</maxRange>
+      <displayRays>true</displayRays>
+    </sensor:ray>
+  </gazebo>
+</xacro:macro>
 <xacro:macro name="kobuki_sim">
   <gazebo>
     <controller:gazebo_ros_kobuki name="kobuki_controller" plugin="libgazebo_ros_kobuki.so">
-      <alwaysOn>true</alwaysOn>
-      <node_namespace>kobuki_node</node_namespace>
-      <left_wheel_joint>wheel_left_joint</left_wheel_joint>
-      <right_wheel_joint>wheel_right_joint</right_wheel_joint>
+      <left_wheel_joint_name>wheel_left_joint</left_wheel_joint_name>
+      <right_wheel_joint_name>wheel_right_joint</right_wheel_joint_name>
       <wheel_separation>.230</wheel_separation>
       <wheel_diameter>0.070</wheel_diameter>
-      <base_geom>base_footprint</base_geom>
-      <updateRate>40</updateRate>
       <torque>1.0</torque>
+      <velocity_command_timeout>0.6</velocity_command_timeout>
+      <cliff_sensor_left_name>cliff_sensor_left</cliff_sensor_left_name>
+      <cliff_sensor_front_name>cliff_sensor_front</cliff_sensor_front_name>
+      <cliff_sensor_right_name>cliff_sensor_right</cliff_sensor_right_name>
+      <cliff_detection_threshold>0.04</cliff_detection_threshold>
+      <bumper_name>bumpers</bumper_name>
+      <base_collision_model_link>base_link</base_collision_model_link>
     </controller:gazebo_ros_kobuki>
   </gazebo>
@@ -24,5 +81,4 @@
     <kp value="100000000.0"/>
     <kd value="10000.0"/>
-    <fdir value="1 0 0"/>
   </gazebo>
   <gazebo reference="wheel_right_link">
@@ -31,5 +87,4 @@
     <kp value="100000000.0"/>
     <kd value="10000.0"/>
-    <fdir value="1 0 0"/>
   </gazebo>
   <gazebo reference="caster_front_link">
@@ -46,52 +101,11 @@
   </gazebo>
 </xacro:macro>
-<xacro:macro name="kobuki_cliff_sensors">
-  <gazebo reference="cliff_sensor_left_link">
-    <sensor:ray name="cliff_sensor_left">
-      <alwaysActive>true</alwaysActive>
-      <rayCount>1</rayCount>
-      <rangeCount>1</rangeCount>
-      <resRange>0.1</resRange>
-      <minAngle>0</minAngle>
-      <maxAngle>0</maxAngle>
-      <minRange>0.01</minRange>
-      <maxRange>0.04</maxRange>
-      <displayRays>false</displayRays>
-    </sensor:ray>
-  </gazebo>
-  <gazebo reference="cliff_sensor_right_link">
-    <sensor:ray name="cliff_sensor_right">
-      <alwaysActive>true</alwaysActive>
-      <rayCount>1</rayCount>
-      <rangeCount>1</rangeCount>
-      <resRange>0.1</resRange>
-      <minAngle>0</minAngle>
-      <maxAngle>0</maxAngle>
-      <minRange>0.01</minRange>
-      <maxRange>0.04</maxRange>
-      <displayRays>false</displayRays>
-    </sensor:ray>
-  </gazebo>
-  <gazebo reference="cliff_sensor_front_link">
-    <sensor:ray name="cliff_sensor_front">
-      <alwaysActive>true</alwaysActive>
-      <rayCount>1</rayCount>
-      <rangeCount>1</rangeCount>
-      <resRange>0.1</resRange>
-      <minAngle>0</minAngle>
-      <maxAngle>0</maxAngle>
-      <minRange>0.01</minRange>
-      <maxRange>0.04</maxRange>
-      <displayRays>false</displayRays>
-    </sensor:ray>
-  </gazebo>
-</xacro:macro>
-<xacro:macro name="turtlebot_sim_imu">
+<xacro:macro name="kobuki_sim_imu">
   <gazebo>
     <controller:gazebo_ros_imu name="imu_controller" plugin="libgazebo_ros_imu.so">
       <alwaysOn>true</alwaysOn>
-      <updateRate>30</updateRate>
+      <updateRate>50</updateRate>
       <bodyName>gyro_link</bodyName>
-      <topicName>imu/data</topicName>
+      <topicName>/mobile_base/sensors/imu_data</topicName>
       <gaussianNoise>${0.0017*0.0017}</gaussianNoise>
       <xyzOffsets>0 0 0</xyzOffsets>

Commit message: kobuki_description: adds a range of small changes to get Kobuki running in Gazebo 1.9+

File: kobuki_description/urdf/kobuki.urdf.xacro (robot description, xacro)
@@ -7,6 +7,6 @@
  -->
 <robot name="kobuki" xmlns:xacro="http://ros.org/wiki/xacro">
-  <include filename="$(find kobuki_description)/urdf/common_properties.urdf.xacro"/>
-  <include filename="$(find kobuki_description)/urdf/kobuki_gazebo.urdf.xacro"/>
+  <xacro:include filename="$(find kobuki_description)/urdf/common_properties.urdf.xacro"/>
+<!--   <xacro:include filename="$(find kobuki_description)/urdf/kobuki_gazebo.urdf.xacro"/> -->
   <!-- Xacro properties -->
   <xacro:property name="M_SCALE" value="0.001"/>
@@ -49,4 +49,6 @@
                  izz="0.0001" />
       </inertial>
+<!--       <kobuki_sim/> -->
+<!--       <kobuki_bumpers/> -->
     </link>
     <joint name="wheel_left_joint" type="continuous">
@@ -159,4 +161,5 @@
                  izz="0.0001"/>
       </inertial>
+<!--       <kobuki_sim_imu/> -->
     </link>
 	  <joint name="cliff_sensor_left_joint" type="fixed">
@@ -173,4 +176,5 @@
                  izz="0.0001" />
       </inertial>
+<!--       <kobuki_cliff_sensor_left/> -->
     </link>
 	  <joint name="cliff_sensor_right_joint" type="fixed">
@@ -187,4 +191,5 @@
                  izz="0.0001" />
       </inertial>
+<!--       <kobuki_cliff_sensor_right/> -->
     </link>
     <joint name="cliff_sensor_front_joint" type="fixed">
@@ -201,10 +206,6 @@
                  izz="0.0001" />
       </inertial>
-    </link>
-    <!--  Gazebo additions -->
-    <kobuki_sim/>
-    <kobuki_bumpers/>
-    <kobuki_cliff_sensors/>
-    <kobuki_sim_imu/>
+<!--       <kobuki_cliff_sensor_front/> -->
+    </link>
   </xacro:macro>
 </robot>

File: kobuki_description/urdf/kobuki_gazebo.urdf.xacro (robot description, xacro)
@@ -1,79 +1,4 @@
 <?xml version="1.0"?>
-<robot xmlns:controller="http://playerstage.sourceforge.net/gazebo/xmlschema/#controller"
-       xmlns:interface="http://playerstage.sourceforge.net/gazebo/xmlschema/#interface"
-       xmlns:sensor="http://playerstage.sourceforge.net/gazebo/xmlschema/#sensor"
-       xmlns:xacro="http://ros.org/wiki/xacro"
-       name="kobuki_gazebo">
-<xacro:macro name="kobuki_bumpers">
-  <gazebo reference="base_link">
-    <sensor:contact name="bumpers">
-      <geom>base_footprint_geom_base_link</geom>
-      <topic>bumpers</topic>
-      <alwaysOn>true</alwaysOn>
-      <updateRate>50</updateRate>
-    </sensor:contact>
-  </gazebo>
-</xacro:macro>
-<xacro:macro name="kobuki_cliff_sensors">
-  <gazebo reference="cliff_sensor_left_link">
-    <sensor:ray name="cliff_sensor_left">
-      <alwaysOn>true</alwaysOn>
-      <updateRate>50</updateRate>
-      <rayCount>50</rayCount>
-      <rangeCount>1</rangeCount>
-      <resRange>1.0</resRange>
-      <minAngle>-0.04361</minAngle>
-      <maxAngle>0.04361</maxAngle>
-      <minRange>0.01</minRange>
-      <maxRange>0.15</maxRange>
-      <displayRays>true</displayRays>
-    </sensor:ray>
-  </gazebo>
-  <gazebo reference="cliff_sensor_right_link">
-    <sensor:ray name="cliff_sensor_right">
-      <alwaysOn>true</alwaysOn>
-      <updateRate>50</updateRate>
-      <rayCount>50</rayCount>
-      <rangeCount>1</rangeCount>
-      <resRange>1.0</resRange>
-      <minAngle>-2.5</minAngle>
-      <maxAngle>2.5</maxAngle>
-      <minRange>0.01</minRange>
-      <maxRange>0.15</maxRange>
-      <displayRays>true</displayRays>
-    </sensor:ray>
-  </gazebo>
-  <gazebo reference="cliff_sensor_front_link">
-    <sensor:ray name="cliff_sensor_front">
-      <alwaysOn>true</alwaysOn>
-      <updateRate>50</updateRate>
-      <rayCount>50</rayCount>
-      <rangeCount>1</rangeCount>
-      <resRange>1.0</resRange>
-      <minAngle>-2.5</minAngle>
-      <maxAngle>2.5</maxAngle>
-      <minRange>0.01</minRange>
-      <maxRange>0.15</maxRange>
-      <displayRays>true</displayRays>
-    </sensor:ray>
-  </gazebo>
-</xacro:macro>
-<xacro:macro name="kobuki_sim">
-  <gazebo>
-    <controller:gazebo_ros_kobuki name="kobuki_controller" plugin="libgazebo_ros_kobuki.so">
-      <left_wheel_joint_name>wheel_left_joint</left_wheel_joint_name>
-      <right_wheel_joint_name>wheel_right_joint</right_wheel_joint_name>
-      <wheel_separation>.230</wheel_separation>
-      <wheel_diameter>0.070</wheel_diameter>
-      <torque>1.0</torque>
-      <velocity_command_timeout>0.6</velocity_command_timeout>
-      <cliff_sensor_left_name>cliff_sensor_left</cliff_sensor_left_name>
-      <cliff_sensor_front_name>cliff_sensor_front</cliff_sensor_front_name>
-      <cliff_sensor_right_name>cliff_sensor_right</cliff_sensor_right_name>
-      <cliff_detection_threshold>0.04</cliff_detection_threshold>
-      <bumper_name>bumpers</bumper_name>
-      <base_collision_model_link>base_link</base_collision_model_link>
-    </controller:gazebo_ros_kobuki>
-  </gazebo>
+<robot>
   <gazebo reference="wheel_left_link">
     <mu1 value="10"/>
@@ -100,8 +25,100 @@
     <kd value="10000.0"/>
   </gazebo>
-</xacro:macro>
-<xacro:macro name="kobuki_sim_imu">
+  <gazebo reference="base_link">
+    <sensor type="contact" name="bumpers">
+      <always_on>1</always_on>
+      <update_rate>50.0</update_rate>
+      <visualize>true</visualize>
+      <contact>
+        <collision>base_footprint_geom_base_link</collision>
+      </contact>
+    </sensor>
+  </gazebo>
+  <gazebo reference="cliff_sensor_left_link">
+    <sensor type="ray" name="cliff_sensor_left">
+      <always_on>true</always_on>
+      <update_rate>50</update_rate>
+      <visualize>true</visualize>
+      <ray>
+        <scan>
+          <horizontal>
+            <samples>50</samples>
+            <resolution>1.0</resolution>
+            <min_angle>-0.0436</min_angle>  <!-- -2.5 degree -->
+            <max_angle>0.0436</max_angle> <!-- 2.5 degree -->
+          </horizontal>
+          <vertical>
+            <samples>50</samples>
+            <resolution>1.0</resolution>
+            <min_angle>-0.0436</min_angle>  <!-- -2.5 degree -->
+            <max_angle>0.0436</max_angle> <!-- 2.5 degree -->
+          </vertical>
+        </scan>
+        <range>
+          <min>0.01</min>
+          <max>0.15</max>
+          <resolution>1.0</resolution>
+        </range>
+      </ray>
+    </sensor>
+  </gazebo>
+  <gazebo reference="cliff_sensor_right_link">
+    <sensor type="ray" name="cliff_sensor_right">
+      <always_on>true</always_on>
+      <update_rate>50</update_rate>
+      <visualize>true</visualize>
+      <ray>
+        <scan>
+          <horizontal>
+            <samples>50</samples>
+            <resolution>1.0</resolution>
+            <min_angle>-0.0436</min_angle>  <!-- -2.5 degree -->
+            <max_angle>0.0436</max_angle> <!-- 2.5 degree -->
+          </horizontal>
+          <vertical>
+            <samples>50</samples>
+            <resolution>1.0</resolution>
+            <min_angle>-0.0436</min_angle>  <!-- -2.5 degree -->
+            <max_angle>0.0436</max_angle> <!-- 2.5 degree -->
+          </vertical>
+        </scan>
+        <range>
+          <min>0.01</min>
+          <max>0.15</max>
+          <resolution>1.0</resolution>
+        </range>
+      </ray>
+    </sensor>
+  </gazebo>
+  <gazebo reference="cliff_sensor_front_link">
+    <sensor type="ray" name="cliff_sensor_front">
+      <always_on>true</always_on>
+      <update_rate>50</update_rate>
+      <visualize>true</visualize>
+      <ray>
+        <scan>
+          <horizontal>
+            <samples>50</samples>
+            <resolution>1.0</resolution>
+            <min_angle>-0.0436</min_angle>  <!-- -2.5 degree -->
+            <max_angle>0.0436</max_angle> <!-- 2.5 degree -->
+          </horizontal>
+          <vertical>
+            <samples>50</samples>
+            <resolution>1.0</resolution>
+            <min_angle>-0.0436</min_angle>  <!-- -2.5 degree -->
+            <max_angle>0.0436</max_angle> <!-- 2.5 degree -->
+          </vertical>
+        </scan>
+        <range>
+          <min>0.01</min>
+          <max>0.15</max>
+          <resolution>1.0</resolution>
+        </range>
+      </ray>
+    </sensor>
+  </gazebo>
   <gazebo>
-    <controller:gazebo_ros_imu name="imu_controller" plugin="libgazebo_ros_imu.so">
+    <plugin name="imu_controller" filename="libgazebo_ros_imu.so">
       <alwaysOn>true</alwaysOn>
       <updateRate>50</updateRate>
@@ -111,7 +128,21 @@
       <xyzOffsets>0 0 0</xyzOffsets>
       <rpyOffsets>0 0 0</rpyOffsets>
-      <interface:position name="gyro_link"/>
-    </controller:gazebo_ros_imu>
+    </plugin>
   </gazebo>
-</xacro:macro>
+  <gazebo>
+    <plugin name="kobuki_controller" filename="libgazebo_ros_kobuki.so">
+      <left_wheel_joint_name>wheel_left_joint</left_wheel_joint_name>
+      <right_wheel_joint_name>wheel_right_joint</right_wheel_joint_name>
+      <wheel_separation>.230</wheel_separation>
+      <wheel_diameter>0.070</wheel_diameter>
+      <torque>1.0</torque>
+      <velocity_command_timeout>0.6</velocity_command_timeout>
+      <cliff_sensor_left_name>cliff_sensor_left</cliff_sensor_left_name>
+      <cliff_sensor_front_name>cliff_sensor_front</cliff_sensor_front_name>
+      <cliff_sensor_right_name>cliff_sensor_right</cliff_sensor_right_name>
+      <cliff_detection_threshold>0.04</cliff_detection_threshold>
+      <bumper_name>bumpers</bumper_name>
+      <base_collision_model_link>base_link</base_collision_model_link>
+    </plugin>
+  </gazebo>
 </robot>

File: kobuki_description/urdf/kobuki_standalone.urdf.xacro (robot description, xacro)
@@ -7,4 +7,5 @@
   <!-- Defines the kobuki component tag. -->
   <include filename="$(find kobuki_description)/urdf/kobuki.urdf.xacro" />
+  <include filename="$(find kobuki_description)/urdf/kobuki_gazebo.urdf.xacro" />
   <kobuki/>
 </robot>
