Commit message: kobuki_description: adds minor changes to gazebo properties

File: kobuki_description/urdf/kobuki.urdf.xacro (robot description, xacro)
@@ -8,7 +8,4 @@
 <robot name="kobuki" xmlns:xacro="http://ros.org/wiki/xacro">
   <xacro:include filename="$(find kobuki_description)/urdf/common_properties.urdf.xacro"/>
-<!--   <xacro:include filename="$(find kobuki_description)/urdf/kobuki_gazebo.urdf.xacro"/> -->
-  <!-- Xacro properties -->
-  <xacro:property name="M_SCALE" value="0.001"/>
   <!-- Kobuki -->
   <xacro:macro name="kobuki">
@@ -43,12 +40,17 @@
       </collision>
       <inertial>
+        <origin xyz="0 0 0"/>
         <mass value="2.4"/> <!-- 2.4/2.6 kg for small/big battery pack -->
-        <origin xyz="0 0 0"/>
-        <inertia ixx="0.0001" ixy="0.0" ixz="0.0"
-                 iyy="0.0001" iyz="0.0"
-                 izz="0.0001" />
-      </inertial>
-<!--       <kobuki_sim/> -->
-<!--       <kobuki_bumpers/> -->
+        <!-- http://en.wikipedia.org/wiki/List_of_moment_of_inertia_tensors
+             Assuming homogeneous mass distribution
+		         m=2.4; h=0.09; r=0.175;
+		         ixx = 1/12*m*(3*r^2 + h^2)
+		         iyy = 1/12*m*(3*r^2 + h^2)
+		         izz = 1/2*m*r^2
+          -->
+        <inertia ixx="0.019995" ixy="0.0" ixz="0.0"
+                 iyy="0.019995" iyz="0.0"
+                 izz="0.006125" />
+      </inertial>
     </link>
     <joint name="wheel_left_joint" type="continuous">
@@ -161,12 +163,11 @@
                  izz="0.0001"/>
       </inertial>
-<!--       <kobuki_sim_imu/> -->
-    </link>
-	  <joint name="cliff_sensor_left_joint" type="fixed">
-	    <origin xyz="0.08734 0.13601 0.0214" rpy="0 ${M_PI/2} 0" />
-	    <parent link="base_link"/>
-	    <child link="cliff_sensor_left_link" />
-	  </joint>
-	  <link name="cliff_sensor_left_link">
+    </link>
+    <joint name="cliff_sensor_left_joint" type="fixed">
+      <origin xyz="0.08734 0.13601 0.0214" rpy="0 ${M_PI/2} 0" />
+      <parent link="base_link"/>
+      <child link="cliff_sensor_left_link" />
+    </joint>
+    <link name="cliff_sensor_left_link">
       <inertial>
         <mass value="0.0001" />
@@ -176,11 +177,10 @@
                  izz="0.0001" />
       </inertial>
-<!--       <kobuki_cliff_sensor_left/> -->
-    </link>
-	  <joint name="cliff_sensor_right_joint" type="fixed">
-	    <origin xyz="0.085 -0.13601 0.0214" rpy="0 ${M_PI/2} 0" />
-	    <parent link="base_link"/>
-	    <child link="cliff_sensor_right_link" />
-	  </joint>
+    </link>
+    <joint name="cliff_sensor_right_joint" type="fixed">
+      <origin xyz="0.085 -0.13601 0.0214" rpy="0 ${M_PI/2} 0" />
+      <parent link="base_link"/>
+      <child link="cliff_sensor_right_link" />
+    </joint>
     <link name="cliff_sensor_right_link">
       <inertial>
@@ -191,5 +191,4 @@
                  izz="0.0001" />
       </inertial>
-<!--       <kobuki_cliff_sensor_right/> -->
     </link>
     <joint name="cliff_sensor_front_joint" type="fixed">
@@ -206,5 +205,4 @@
                  izz="0.0001" />
       </inertial>
-<!--       <kobuki_cliff_sensor_front/> -->
     </link>
   </xacro:macro>

File: kobuki_description/urdf/kobuki_gazebo.urdf.xacro (robot description, xacro)
@@ -2,26 +2,26 @@
 <robot>
   <gazebo reference="wheel_left_link">
-    <mu1 value="10"/>
-    <mu2 value="10"/>
-    <kp value="100000000.0"/>
-    <kd value="10000.0"/>
+    <mu1>1.0</mu1>
+    <mu2>1.0</mu2>
+    <kp>100000000.0</kp>
+    <kd>10000.0</kd>
   </gazebo>
   <gazebo reference="wheel_right_link">
-    <mu1 value="10"/>
-    <mu2 value="10"/>
-    <kp value="100000000.0"/>
-    <kd value="10000.0"/>
+    <mu1>1.0</mu1>
+    <mu2>1.0</mu2>
+    <kp>100000000.0</kp>
+    <kd>10000.0</kd>
   </gazebo>
   <gazebo reference="caster_front_link">
-    <mu1 value="0"/>
-    <mu2 value="0"/>
-    <kp value="100000000.0"/>
-    <kd value="10000.0"/>
+    <mu1>0.0</mu1>
+    <mu2>0.0</mu2>
+    <kp>100000000.0</kp>
+    <kd>10000.0</kd>
   </gazebo>
   <gazebo reference="caster_back_link">
-    <mu1 value="0"/>
-    <mu2 value="0"/>
-    <kp value="100000000.0"/>
-    <kd value="10000.0"/>
+    <mu1>0.0</mu1>
+    <mu2>0.0</mu2>
+    <kp>100000000.0</kp>
+    <kd>10000.0</kd>
   </gazebo>
   <gazebo reference="base_link">

Commit message: adds another Gazebo related fix

File: kobuki_description/urdf/kobuki.urdf.xacro (robot description, xacro)
@@ -207,4 +207,6 @@
       </inertial>
     </link>
+    <!-- Kobuki Gazebo simulation details -->
+    <kobuki_sim/>
   </xacro:macro>
 </robot>

File: kobuki_description/urdf/kobuki_gazebo.urdf.xacro (robot description, xacro)
@@ -1,150 +1,152 @@
 <?xml version="1.0"?>
-<robot>
-  <gazebo reference="wheel_left_link">
-    <mu1>1.0</mu1>
-    <mu2>1.0</mu2>
-    <kp>100000000.0</kp>
-    <kd>10000.0</kd>
-  </gazebo>
-  <gazebo reference="wheel_right_link">
-    <mu1>1.0</mu1>
-    <mu2>1.0</mu2>
-    <kp>100000000.0</kp>
-    <kd>10000.0</kd>
-  </gazebo>
-  <gazebo reference="caster_front_link">
-    <mu1>0.0</mu1>
-    <mu2>0.0</mu2>
-    <kp>100000000.0</kp>
-    <kd>10000.0</kd>
-  </gazebo>
-  <gazebo reference="caster_back_link">
-    <mu1>0.0</mu1>
-    <mu2>0.0</mu2>
-    <kp>100000000.0</kp>
-    <kd>10000.0</kd>
-  </gazebo>
-  <gazebo reference="base_link">
-    <sensor type="contact" name="bumpers">
-      <always_on>1</always_on>
-      <update_rate>50.0</update_rate>
-      <visualize>true</visualize>
-      <contact>
-        <collision>base_footprint_geom_base_link</collision>
-      </contact>
-    </sensor>
-  </gazebo>
-  <gazebo reference="cliff_sensor_left_link">
-    <sensor type="ray" name="cliff_sensor_left">
-      <always_on>true</always_on>
-      <update_rate>50</update_rate>
-      <visualize>true</visualize>
-      <ray>
-        <scan>
-          <horizontal>
-            <samples>50</samples>
-            <resolution>1.0</resolution>
-            <min_angle>-0.0436</min_angle>  <!-- -2.5 degree -->
-            <max_angle>0.0436</max_angle> <!-- 2.5 degree -->
-          </horizontal>
-          <vertical>
-            <samples>50</samples>
-            <resolution>1.0</resolution>
-            <min_angle>-0.0436</min_angle>  <!-- -2.5 degree -->
-            <max_angle>0.0436</max_angle> <!-- 2.5 degree -->
-          </vertical>
-        </scan>
-        <range>
-          <min>0.01</min>
-          <max>0.15</max>
-          <resolution>1.0</resolution>
-        </range>
-      </ray>
-    </sensor>
-  </gazebo>
-  <gazebo reference="cliff_sensor_right_link">
-    <sensor type="ray" name="cliff_sensor_right">
-      <always_on>true</always_on>
-      <update_rate>50</update_rate>
-      <visualize>true</visualize>
-      <ray>
-        <scan>
-          <horizontal>
-            <samples>50</samples>
-            <resolution>1.0</resolution>
-            <min_angle>-0.0436</min_angle>  <!-- -2.5 degree -->
-            <max_angle>0.0436</max_angle> <!-- 2.5 degree -->
-          </horizontal>
-          <vertical>
-            <samples>50</samples>
-            <resolution>1.0</resolution>
-            <min_angle>-0.0436</min_angle>  <!-- -2.5 degree -->
-            <max_angle>0.0436</max_angle> <!-- 2.5 degree -->
-          </vertical>
-        </scan>
-        <range>
-          <min>0.01</min>
-          <max>0.15</max>
-          <resolution>1.0</resolution>
-        </range>
-      </ray>
-    </sensor>
-  </gazebo>
-  <gazebo reference="cliff_sensor_front_link">
-    <sensor type="ray" name="cliff_sensor_front">
-      <always_on>true</always_on>
-      <update_rate>50</update_rate>
-      <visualize>true</visualize>
-      <ray>
-        <scan>
-          <horizontal>
-            <samples>50</samples>
-            <resolution>1.0</resolution>
-            <min_angle>-0.0436</min_angle>  <!-- -2.5 degree -->
-            <max_angle>0.0436</max_angle> <!-- 2.5 degree -->
-          </horizontal>
-          <vertical>
-            <samples>50</samples>
-            <resolution>1.0</resolution>
-            <min_angle>-0.0436</min_angle>  <!-- -2.5 degree -->
-            <max_angle>0.0436</max_angle> <!-- 2.5 degree -->
-          </vertical>
-        </scan>
-        <range>
-          <min>0.01</min>
-          <max>0.15</max>
-          <resolution>1.0</resolution>
-        </range>
-      </ray>
-    </sensor>
-  </gazebo>
-  <gazebo>
-    <plugin name="imu_controller" filename="libgazebo_ros_imu.so">
-      <alwaysOn>true</alwaysOn>
-      <updateRate>50</updateRate>
-      <bodyName>gyro_link</bodyName>
-      <topicName>/mobile_base/sensors/imu_data</topicName>
-      <serviceName>imu/is_calibrated</serviceName>
-      <gaussianNoise>${0.0017*0.0017}</gaussianNoise>
-      <xyzOffsets>0 0 0</xyzOffsets>
-      <rpyOffsets>0 0 0</rpyOffsets>
-    </plugin>
-  </gazebo>
-  <gazebo>
-    <plugin name="kobuki_controller" filename="libgazebo_ros_kobuki.so">
-      <publish_tf>0</publish_tf>
-      <left_wheel_joint_name>wheel_left_joint</left_wheel_joint_name>
-      <right_wheel_joint_name>wheel_right_joint</right_wheel_joint_name>
-      <wheel_separation>.230</wheel_separation>
-      <wheel_diameter>0.070</wheel_diameter>
-      <torque>1.0</torque>
-      <velocity_command_timeout>0.6</velocity_command_timeout>
-      <cliff_sensor_left_name>cliff_sensor_left</cliff_sensor_left_name>
-      <cliff_sensor_front_name>cliff_sensor_front</cliff_sensor_front_name>
-      <cliff_sensor_right_name>cliff_sensor_right</cliff_sensor_right_name>
-      <cliff_detection_threshold>0.04</cliff_detection_threshold>
-      <bumper_name>bumpers</bumper_name>
-      <base_collision_model_link>base_link</base_collision_model_link>
-    </plugin>
-  </gazebo>
+<robot name="kobuki_sim" xmlns:xacro="http://ros.org/wiki/xacro">
+  <xacro:macro name="kobuki_sim">
+	  <gazebo reference="wheel_left_link">
+	    <mu1>1.0</mu1>
+	    <mu2>1.0</mu2>
+	    <kp>100000000.0</kp>
+	    <kd>10000.0</kd>
+	  </gazebo>
+	  <gazebo reference="wheel_right_link">
+	    <mu1>1.0</mu1>
+	    <mu2>1.0</mu2>
+	    <kp>100000000.0</kp>
+	    <kd>10000.0</kd>
+	  </gazebo>
+	  <gazebo reference="caster_front_link">
+	    <mu1>0.0</mu1>
+	    <mu2>0.0</mu2>
+	    <kp>100000000.0</kp>
+	    <kd>10000.0</kd>
+	  </gazebo>
+	  <gazebo reference="caster_back_link">
+	    <mu1>0.0</mu1>
+	    <mu2>0.0</mu2>
+	    <kp>100000000.0</kp>
+	    <kd>10000.0</kd>
+	  </gazebo>
+	  <gazebo reference="base_link">
+	    <sensor type="contact" name="bumpers">
+	      <always_on>1</always_on>
+	      <update_rate>50.0</update_rate>
+	      <visualize>true</visualize>
+	      <contact>
+	        <collision>base_footprint_geom_base_link</collision>
+	      </contact>
+	    </sensor>
+	  </gazebo>
+	  <gazebo reference="cliff_sensor_left_link">
+	    <sensor type="ray" name="cliff_sensor_left">
+	      <always_on>true</always_on>
+	      <update_rate>50</update_rate>
+	      <visualize>true</visualize>
+	      <ray>
+	        <scan>
+	          <horizontal>
+	            <samples>50</samples>
+	            <resolution>1.0</resolution>
+	            <min_angle>-0.0436</min_angle>  <!-- -2.5 degree -->
+	            <max_angle>0.0436</max_angle> <!-- 2.5 degree -->
+	          </horizontal>
+	          <vertical>
+	            <samples>50</samples>
+	            <resolution>1.0</resolution>
+	            <min_angle>-0.0436</min_angle>  <!-- -2.5 degree -->
+	            <max_angle>0.0436</max_angle> <!-- 2.5 degree -->
+	          </vertical>
+	        </scan>
+	        <range>
+	          <min>0.01</min>
+	          <max>0.15</max>
+	          <resolution>1.0</resolution>
+	        </range>
+	      </ray>
+	    </sensor>
+	  </gazebo>
+	  <gazebo reference="cliff_sensor_right_link">
+	    <sensor type="ray" name="cliff_sensor_right">
+	      <always_on>true</always_on>
+	      <update_rate>50</update_rate>
+	      <visualize>true</visualize>
+	      <ray>
+	        <scan>
+	          <horizontal>
+	            <samples>50</samples>
+	            <resolution>1.0</resolution>
+	            <min_angle>-0.0436</min_angle>  <!-- -2.5 degree -->
+	            <max_angle>0.0436</max_angle> <!-- 2.5 degree -->
+	          </horizontal>
+	          <vertical>
+	            <samples>50</samples>
+	            <resolution>1.0</resolution>
+	            <min_angle>-0.0436</min_angle>  <!-- -2.5 degree -->
+	            <max_angle>0.0436</max_angle> <!-- 2.5 degree -->
+	          </vertical>
+	        </scan>
+	        <range>
+	          <min>0.01</min>
+	          <max>0.15</max>
+	          <resolution>1.0</resolution>
+	        </range>
+	      </ray>
+	    </sensor>
+	  </gazebo>
+	  <gazebo reference="cliff_sensor_front_link">
+	    <sensor type="ray" name="cliff_sensor_front">
+	      <always_on>true</always_on>
+	      <update_rate>50</update_rate>
+	      <visualize>true</visualize>
+	      <ray>
+	        <scan>
+	          <horizontal>
+	            <samples>50</samples>
+	            <resolution>1.0</resolution>
+	            <min_angle>-0.0436</min_angle>  <!-- -2.5 degree -->
+	            <max_angle>0.0436</max_angle> <!-- 2.5 degree -->
+	          </horizontal>
+	          <vertical>
+	            <samples>50</samples>
+	            <resolution>1.0</resolution>
+	            <min_angle>-0.0436</min_angle>  <!-- -2.5 degree -->
+	            <max_angle>0.0436</max_angle> <!-- 2.5 degree -->
+	          </vertical>
+	        </scan>
+	        <range>
+	          <min>0.01</min>
+	          <max>0.15</max>
+	          <resolution>1.0</resolution>
+	        </range>
+	      </ray>
+	    </sensor>
+	  </gazebo>
+	  <gazebo>
+	    <plugin name="imu_controller" filename="libgazebo_ros_imu.so">
+	      <alwaysOn>true</alwaysOn>
+	      <updateRate>50</updateRate>
+	      <bodyName>gyro_link</bodyName>
+	      <topicName>/mobile_base/sensors/imu_data</topicName>
+	      <serviceName>imu/is_calibrated</serviceName>
+	      <gaussianNoise>${0.0017*0.0017}</gaussianNoise>
+	      <xyzOffsets>0 0 0</xyzOffsets>
+	      <rpyOffsets>0 0 0</rpyOffsets>
+	    </plugin>
+	  </gazebo>
+	  <gazebo>
+	    <plugin name="kobuki_controller" filename="libgazebo_ros_kobuki.so">
+	      <publish_tf>0</publish_tf>
+	      <left_wheel_joint_name>wheel_left_joint</left_wheel_joint_name>
+	      <right_wheel_joint_name>wheel_right_joint</right_wheel_joint_name>
+	      <wheel_separation>.230</wheel_separation>
+	      <wheel_diameter>0.070</wheel_diameter>
+	      <torque>1.0</torque>
+	      <velocity_command_timeout>0.6</velocity_command_timeout>
+	      <cliff_sensor_left_name>cliff_sensor_left</cliff_sensor_left_name>
+	      <cliff_sensor_front_name>cliff_sensor_front</cliff_sensor_front_name>
+	      <cliff_sensor_right_name>cliff_sensor_right</cliff_sensor_right_name>
+	      <cliff_detection_threshold>0.04</cliff_detection_threshold>
+	      <bumper_name>bumpers</bumper_name>
+	      <base_collision_model_link>base_link</base_collision_model_link>
+	    </plugin>
+	  </gazebo>
+  </xacro:macro>
 </robot>

Commit message: corrects inertia and center of mass using an approximation (fixes #271)

File: kobuki_description/urdf/kobuki.urdf.xacro (robot description, xacro)
@@ -41,16 +41,17 @@
       </collision>
       <inertial>
-        <origin xyz="0 0 0"/>
+        <!-- COM experimentally determined -->
+        <origin xyz="0.01 0 0"/>
         <mass value="2.4"/> <!-- 2.4/2.6 kg for small/big battery pack -->
-        <!-- http://en.wikipedia.org/wiki/List_of_moment_of_inertia_tensors
-             Assuming homogeneous mass distribution
-		         m=2.4; h=0.09; r=0.175;
-		         ixx = 1/12*m*(3*r^2 + h^2)
-		         iyy = 1/12*m*(3*r^2 + h^2)
-		         izz = 1/2*m*r^2
+        <!-- Kobuki's inertia tensor is approximated by a cylinder with homogeneous mass distribution
+             More details: http://en.wikipedia.org/wiki/List_of_moment_of_inertia_tensors
+             m = 2.4 kg; h = 0.09 m; r = 0.175 m
+             ixx = 1/12 * m * (3 * r^2 + h^2)
+             iyy = 1/12 * m * (3 * r^2 + h^2)
+             izz = 1/2 * m * r^2
           -->
         <inertia ixx="0.019995" ixy="0.0" ixz="0.0"
                  iyy="0.019995" iyz="0.0"
-                 izz="0.006125" />
+                 izz="0.03675" />
       </inertial>
     </link>

Commit message: [description] collision box naming changed with kinetic's gazebo
This redirects it properly. Also some whitespacing updates.

File: kobuki_description/urdf/kobuki.urdf.xacro (robot description, xacro)
@@ -34,5 +34,5 @@
         <origin xyz="0.001 0 0.05199" rpy="0 0 0"/>
       </visual>
-      <collision>
+      <collision name="base">
         <geometry>
           <cylinder length="0.10938" radius="0.178"/>

File: kobuki_description/urdf/kobuki_gazebo.urdf.xacro (robot description, xacro)
@@ -42,5 +42,5 @@
 	      <visualize>true</visualize>
 	      <contact>
-	        <collision>base_footprint_collision_base_link</collision>
+	        <collision>base_footprint_fixed_joint_lump__base_collision</collision>
 	      </contact>
 	    </sensor>

Commit message: Fix #400: set both wheels to 35mm
Thanks to @gavanderhoorn  for the catch!

File: kobuki_description/urdf/kobuki.urdf.xacro (robot description, xacro)
@@ -71,5 +71,5 @@
       <collision>
         <geometry>
-          <cylinder length="0.0206" radius="0.0352"/>
+          <cylinder length="0.0206" radius="0.035"/>
         </geometry>
         <origin rpy="0 0 0" xyz="0 0 0"/>
@@ -98,5 +98,5 @@
       <collision>
         <geometry>
-          <cylinder length="0.0206" radius="0.0350"/>
+          <cylinder length="0.0206" radius="0.035"/>
         </geometry>
         <origin rpy="0 0 0" xyz="0 0 0"/>
